File: MegaCD-837-8952-Export/MegaCD.kicad_sch (KiCad schematic)
At the start: 184 parts, among them CN1 CON 25P ANGLE, CN2 EDGE 60P, CN3 CON 21P, IC1 68HC000, IC10 65256BLFP-10T, IC11 65256BLFP-10T, IC12 74HC86, IC13 LC8951, IC14 MB8464A-90L, IC15 MB8464A-90L, IC16 MB8464A-10L, IC17 74AC74, IC2 315-5548/315-5632, IC3 315-5476A, IC4 27C1024, IC5 HM514270, IC6 MB3790, IC7 TC511664BZ, IC8 TC511664BZ, IC9 74HC245, J2 2TS, J3 MH, J4 CAS0, M0 TestPoint, M1 TestPoint, M10 TestPoint, M11 TestPoint, M12 TestPoint, M13 TestPoint, M14 TestPoint, M192 TestPoint, M2 TestPoint, M3 TestPoint, M4 TestPoint, M5 TestPoint, M57 TestPoint, M6 TestPoint, M7 TestPoint, M8 TestPoint, M9 TestPoint

Commit message: Minor tweaks
Parts:
- JF1: value 64K -> 8K
- JF2: value 256K -> 32K
Other:
- moved on the sheet: JF1, M0
Changed lines of the file:
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@@
   (junction (at 684.53 115.57) (diameter 0) (color 0 0 0 0)
   )
-  (junction (at 111.76 63.5) (diameter 0) (color 0 0 0 0)
-  )
   (junction (at 265.43 461.01) (diameter 0) (color 0 0 0 0)
   )
@@
   (junction (at 320.04 535.94) (diameter 0) (color 0 0 0 0)
   )
-  (junction (at 129.54 63.5) (diameter 0) (color 0 0 0 0)
-  )
   (junction (at 57.15 563.88) (diameter 0) (color 0 0 0 0)
   )
@@
   (junction (at 264.16 243.84) (diameter 0) (color 0 0 0 0)
   )
-  (junction (at 116.84 63.5) (diameter 0) (color 0 0 0 0)
+  (junction (at 113.03 63.5) (diameter 0) (color 0 0 0 0)
   )
   (junction (at 92.71 231.14) (diameter 0) (color 0 0 0 0)
@@
   (junction (at 734.06 189.23) (diameter 0) (color 0 0 0 0)
   )
+  (junction (at 128.27 63.5) (diameter 0) (color 0 0 0 0)
+  )
   (junction (at 179.07 528.32) (diameter 0) (color 0 0 0 0)
   )
@@
   (junction (at 173.99 486.41) (diameter 0) (color 0 0 0 0)
   )
+  (junction (at 125.73 63.5) (diameter 0) (color 0 0 0 0)
+  )
   (junction (at 632.46 53.34) (diameter 0) (color 0 0 0 0)
   )
@@
     (stroke (width 0) (type default))
   )
-  (bus_entry (at 137.16 73.66) (size 2.54 -2.54)
+  (bus_entry (at 139.7 53.34) (size -2.54 -2.54)
     (stroke (width 0) (type default))
   )
@@
     (stroke (width 0) (type default))
   )
+  (wire (pts (xy 107.95 63.5) (xy 113.03 63.5))
+    (stroke (width 0) (type default))
+  )
   (wire (pts (xy 229.87 435.61) (xy 229.87 430.53))
     (stroke (width 0) (type default))
@@
     (stroke (width 0) (type default))
   )
+  (wire (pts (xy 125.73 63.5) (xy 124.46 63.5))
+    (stroke (width 0) (type default))
+  )
   (wire (pts (xy 243.84 85.09) (xy 255.27 85.09))
     (stroke (width 0) (type default))
@@
     (stroke (width 0) (type default))
   )
+  (bus (pts (xy 137.16 50.8) (xy 137.16 22.86))
+    (stroke (width 0) (type default))
+  )
   (wire (pts (xy 650.24 207.01) (xy 679.45 207.01))
     (stroke (width 0) (type default))
@@
     (stroke (width 0) (type default))
   )
+  (wire (pts (xy 113.03 67.31) (xy 125.73 67.31))
+    (stroke (width 0) (type default))
+  )
   (wire (pts (xy 139.7 121.92) (xy 151.13 121.92))
     (stroke (width 0) (type default))
@@
     (stroke (width 0) (type default))
   )
-  (wire (pts (xy 139.7 71.12) (xy 156.21 71.12))
+  (wire (pts (xy 139.7 53.34) (xy 156.21 53.34))
     (stroke (width 0) (type default))
   )
@@
     (stroke (width 0) (type default))
   )
-  (wire (pts (xy 129.54 63.5) (xy 134.62 63.5))
+  (wire (pts (xy 125.73 63.5) (xy 128.27 63.5))
     (stroke (width 0) (type default))
   )
@@
     (stroke (width 0) (type default))
   )
-  (wire (pts (xy 111.76 66.04) (xy 111.76 63.5))
+  (wire (pts (xy 128.27 58.42) (xy 128.27 63.5))
     (stroke (width 0) (type default))
   )
@@
     (stroke (width 0) (type default))
   )
+  (wire (pts (xy 128.27 63.5) (xy 134.62 63.5))
+    (stroke (width 0) (type default))
+  )
   (wire (pts (xy 457.2 554.99) (xy 462.28 554.99))
     (stroke (width 0) (type default))
@@
     (stroke (width 0) (type default))
   )
-  (wire (pts (xy 116.84 63.5) (xy 116.84 67.31))
+  (wire (pts (xy 113.03 63.5) (xy 113.03 67.31))
     (stroke (width 0) (type default))
   )
@@
     (stroke (width 0) (type default))
   )
-  (bus (pts (xy 137.16 104.14) (xy 137.16 73.66))
+  (bus (pts (xy 137.16 50.8) (xy 137.16 104.14))
     (stroke (width 0) (type default))
   )
@@
     (stroke (width 0) (type default))
   )
-  (wire (pts (xy 107.95 63.5) (xy 111.76 63.5))
-    (stroke (width 0) (type default))
-  )
   (wire (pts (xy 267.97 175.26) (xy 267.97 135.89))
     (stroke (width 0) (type default))
@@
     (stroke (width 0) (type default))
   )
-  (wire (pts (xy 111.76 63.5) (xy 116.84 63.5))
-    (stroke (width 0) (type default))
-  )
   (wire (pts (xy 264.16 553.72) (xy 264.16 563.88))
     (stroke (width 0) (type default))
@@
     (stroke (width 0) (type default))
   )
-  (wire (pts (xy 128.27 63.5) (xy 129.54 63.5))
-    (stroke (width 0) (type default))
-  )
   (bus (pts (xy 679.45 321.31) (xy 679.45 323.85))
     (stroke (width 0) (type default))
@@
     (stroke (width 0) (type default))
   )
-  (wire (pts (xy 156.21 71.12) (xy 156.21 63.5))
+  (wire (pts (xy 156.21 53.34) (xy 156.21 63.5))
     (stroke (width 0) (type default))
   )
@@
     (stroke (width 0) (type default))
   )
-  (wire (pts (xy 116.84 63.5) (xy 118.11 63.5))
+  (wire (pts (xy 113.03 63.5) (xy 114.3 63.5))
     (stroke (width 0) (type default))
   )
@@
     (stroke (width 0) (type default))
   )
-  (wire (pts (xy 129.54 67.31) (xy 129.54 63.5))
+  (wire (pts (xy 125.73 67.31) (xy 125.73 63.5))
     (stroke (width 0) (type default))
   )
@@
     (stroke (width 0) (type default))
   )
-  (bus (pts (xy 137.16 73.66) (xy 137.16 22.86))
-    (stroke (width 0) (type default))
-  )
   (bus (pts (xy 257.81 321.31) (xy 257.81 323.85))
     (stroke (width 0) (type default))
@@
     (stroke (width 0) (type default))
   )
-  (wire (pts (xy 116.84 67.31) (xy 129.54 67.31))
-    (stroke (width 0) (type default))
-  )
   (bus (pts (xy 132.08 144.78) (xy 132.08 142.24))
     (stroke (width 0) (type default))
@@
     (effects (font (size 1.27 1.27)) (justify left bottom))
   )
-  (label "A14" (at 144.78 71.12 0) (fields_autoplaced)
+  (label "A14" (at 144.78 53.34 0) (fields_autoplaced)
     (effects (font (size 1.27 1.27)) (justify left bottom))
   )
@@
     )
   )
-  (symbol (lib_id "Jumper:Jumper_2_Bridged") (at 123.19 63.5 0) (unit 1)
+  (symbol (lib_id "Jumper:Jumper_2_Bridged") (at 119.38 63.5 0) (unit 1)
     (in_bom yes) (on_board yes) (dnp no)
-    (property "Reference" "JF1" (at 123.19 57.15 0)
+    (property "Reference" "JF1" (at 119.38 57.15 0)
       (effects (font (size 1.27 1.27)))
     )
-    (property "Value" "64K" (at 123.19 59.69 0)
+    (property "Value" "8K" (at 119.38 59.69 0)
       (effects (font (size 1.27 1.27)))
     )
-    (property "Footprint" "MegaCD_Footprints:SMD_0805_HandSolder" (at 123.19 63.5 0)
+    (property "Footprint" "MegaCD_Footprints:SMD_0805_HandSolder" (at 119.38 63.5 0)
       (effects (font (size 1.27 1.27)) hide)
     )
-    (property "Datasheet" "~" (at 123.19 63.5 0)
+    (property "Datasheet" "~" (at 119.38 63.5 0)
       (effects (font (size 1.27 1.27)) hide)
     )
@@
     )
   )
-  (symbol (lib_id "Connector:TestPoint") (at 111.76 66.04 180) (unit 1)
+  (symbol (lib_id "Connector:TestPoint") (at 128.27 58.42 0) (unit 1)
     (in_bom yes) (on_board yes) (dnp no)
-    (property "Reference" "M0" (at 112.395 71.12 90)
+    (property "Reference" "M0" (at 127.635 53.34 90)
       (effects (font (size 1.27 1.27)) (justify left))
     )
-    (property "Value" "TestPoint" (at 109.855 71.12 90)
+    (property "Value" "TestPoint" (at 130.175 53.34 90)
       (effects (font (size 1.27 1.27)) (justify left))
     )
-    (property "Footprint" "MegaCD_Footprints:Test_Point_1.5mm" (at 106.68 66.04 0)
+    (property "Footprint" "MegaCD_Footprints:Test_Point_1.5mm" (at 133.35 58.42 0)
       (effects (font (size 1.27 1.27)) hide)
     )
-    (property "Datasheet" "~" (at 106.68 66.04 0)
+    (property "Datasheet" "~" (at 133.35 58.42 0)
       (effects (font (size 1.27 1.27)) hide)
     )
@@
       (effects (font (size 1.27 1.27)))
     )
-    (property "Value" "256K" (at 146.05 59.69 0)
+    (property "Value" "32K" (at 146.05 59.69 0)
       (effects (font (size 1.27 1.27)))
     )
