File: MegaCD-837-8952-Export/MegaCD.kicad_sch (KiCad schematic)
At the start: 184 parts, among them CN1 CON 25P ANGLE, CN2 EDGE 60P, CN3 CON 21P, IC1 68HC000, IC10 65256BLFP-10T, IC11 65256BLFP-10T, IC12 74HC86, IC13 LC8951, IC14 MB8464A-90L, IC15 MB8464A-90L, IC16 MB8464A-10L, IC17 74AC74, IC2 315-5548/315-5632, IC3 315-5476A, IC4 27C1024, IC5 HM514270, IC6 MB3790, IC7 TC511664BZ, IC8 TC511664BZ, IC9 74HC245, J2 2TS, J3 MH, J4 CAS0, M0 TestPoint, M1 TestPoint, M10 TestPoint, M11 TestPoint, M12 TestPoint, M13 TestPoint, M14 TestPoint, M192 TestPoint, M2 TestPoint, M3 TestPoint, M4 TestPoint, M5 TestPoint, M57 TestPoint, M6 TestPoint, M7 TestPoint, M8 TestPoint, M9 TestPoint

Commit message: I forget, probably something incredibly important.
Parts:
- added JF3: A15, MegaCD_Footprints:SMD_0805_HandSolder, symbol Jumper:Jumper_2_Open
Connections:
- net A15: now also JF3.1 (A); no longer IC16.1 (N.C./A14)
- new net: IC16.1 (N.C./A14), JF3.2 (B)
Changed lines of the file:
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@@
     (stroke (width 0) (type default))
   )
-  (bus_entry (at 137.16 154.94) (size 2.54 2.54)
+  (bus_entry (at 137.16 167.64) (size 2.54 2.54)
     (stroke (width 0) (type default))
   )
@@
     (stroke (width 0) (type default))
   )
+  (wire (pts (xy 139.7 170.18) (xy 143.51 170.18))
+    (stroke (width 0) (type default))
+  )
   (wire (pts (xy 519.43 281.94) (xy 519.43 293.37))
     (stroke (width 0) (type default))
@@
     (stroke (width 0) (type default))
   )
+  (wire (pts (xy 153.67 170.18) (xy 156.21 170.18))
+    (stroke (width 0) (type default))
+  )
   (wire (pts (xy 256.54 102.87) (xy 245.11 102.87))
     (stroke (width 0) (type default))
@@
     (stroke (width 0) (type default))
   )
-  (bus (pts (xy 137.16 134.62) (xy 137.16 154.94))
+  (bus (pts (xy 137.16 134.62) (xy 137.16 167.64))
     (stroke (width 0) (type default))
   )
@@
     (stroke (width 0) (type default))
   )
+  (wire (pts (xy 147.32 162.56) (xy 147.32 157.48))
+    (stroke (width 0) (type default))
+  )
   (wire (pts (xy 74.93 483.87) (xy 74.93 462.28))
     (stroke (width 0) (type default))
@@
     (stroke (width 0) (type default))
   )
-  (wire (pts (xy 139.7 157.48) (xy 149.86 157.48))
-    (stroke (width 0) (type default))
-  )
   (wire (pts (xy 345.44 160.02) (xy 336.55 160.02))
     (stroke (width 0) (type default))
@@
     (stroke (width 0) (type default))
   )
+  (wire (pts (xy 156.21 170.18) (xy 156.21 162.56))
+    (stroke (width 0) (type default))
+  )
   (wire (pts (xy 472.44 554.99) (xy 469.9 554.99))
     (stroke (width 0) (type default))
@@
     (stroke (width 0) (type default))
   )
+  (wire (pts (xy 156.21 162.56) (xy 147.32 162.56))
+    (stroke (width 0) (type default))
+  )
   (wire (pts (xy 264.16 553.72) (xy 264.16 563.88))
     (stroke (width 0) (type default))
@@
     (stroke (width 0) (type default))
   )
+  (wire (pts (xy 147.32 157.48) (xy 149.86 157.48))
+    (stroke (width 0) (type default))
+  )
   (bus (pts (xy 45.72 285.75) (xy 45.72 303.53))
     (stroke (width 0) (type default))
@@
     (effects (font (size 1.27 1.27)) (justify right bottom))
   )
-  (label "A15" (at 144.78 157.48 0) (fields_autoplaced)
+  (label "A15" (at 140.97 170.18 0) (fields_autoplaced)
     (effects (font (size 1.27 1.27)) (justify left bottom))
   )
@@
         )
       )
+    )
+  )
+  (symbol (lib_id "Jumper:Jumper_2_Open") (at 148.59 170.18 0) (unit 1)
+    (in_bom yes) (on_board yes) (dnp no)
+    (property "Reference" "JF3" (at 148.59 172.72 0)
+      (effects (font (size 1.27 1.27)))
+    )
+    (property "Value" "A15" (at 148.59 175.26 0)
+      (effects (font (size 1.27 1.27)))
+    )
+    (property "Footprint" "MegaCD_Footprints:SMD_0805_HandSolder" (at 148.59 170.18 0)
+      (effects (font (size 1.27 1.27)) hide)
+    )
+    (property "Datasheet" "~" (at 148.59 170.18 0)
+      (effects (font (size 1.27 1.27)) hide)
+    )
+    (property "Sim.Enable" "0" (at 148.59 170.18 0)
+      (effects (font (size 1.27 1.27)) hide)
+    )
+    (pin "1")
+    (pin "2")
+    (instances
+      (project "MegaCD"
+        (path "/0cd008a0-ed23-4303-a3f0-e3f038adfe31"
+          (reference "JF3") (unit 1)
+        )
+      )
