File: MegaCD-837-8015-Rev0-MCE1/MegaCD.kicad_sch (KiCad schematic)
At the start: 126 parts, among them CN1 CON 25P ANGLE, CN2 EDGE 60P, CN3 CON 21P, IC1 68HC000, IC10 MB8464A-10L, IC11 TC511664BZ, IC12 TC511664BZ, IC13 65256BLFP-10T, IC14 65256BLFP-10T, IC15 LC8951, IC16 74HC00, IC17 MB8464A-90L, IC18 MB8464A-90L, IC19 74HC112, IC2 315-5477, IC20 74HC245, IC3 315-5476, IC4 27C1024, IC5 MB81C4256Z, IC5678 HM514270, IC6 MB81C4256Z, IC7 MB81C4256Z, IC8 MB81C4256Z, IC9 MB3790, J2 2TS, J3 MH, J4 CAS0, M0 TestPoint, M1 TestPoint, M10 TestPoint, M11 TestPoint, M2 TestPoint, M3 TestPoint, M4 TestPoint, M5 TestPoint, M6 TestPoint, M7 TestPoint, M8 TestPoint, M9 TestPoint

Commit message: Mark symbols that are not used more consistently
Parts:
- C15, C16, C17, C18, C19, C20, C21, C22: value 0 -> Not used
- C47: value 200pF -> Not used
- C55: value 33pF -> Not used
- C5678: value 5678uF -> Not used
- CY49, CY50: value 22nF -> Not used
Changed lines of the file:
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@@
       (effects (font (size 1.27 1.27)) (justify left))
     )
-    (property "Value" "0" (at 241.3 73.66 90)
+    (property "Value" "Not used" (at 241.3 73.66 90)
       (effects (font (size 1.27 1.27)) (justify left))
     )
@@
       (effects (font (size 1.27 1.27)) (justify left))
     )
-    (property "Value" "0" (at 232.41 73.66 90)
+    (property "Value" "Not used" (at 232.41 73.66 90)
       (effects (font (size 1.27 1.27)) (justify left))
     )
@@
       (effects (font (size 1.27 1.27)) (justify left))
     )
-    (property "Value" "22nF" (at 260.35 552.45 0)
+    (property "Value" "Not used" (at 260.35 552.45 0)
       (effects (font (size 1.27 1.27)) (justify left))
     )
@@
       (effects (font (size 1.27 1.27)) (justify left))
     )
-    (property "Value" "22nF" (at 217.17 553.72 0)
+    (property "Value" "Not used" (at 217.17 553.72 0)
       (effects (font (size 1.27 1.27)) (justify left))
     )
@@
       (effects (font (size 1.27 1.27)) (justify left))
     )
-    (property "Value" "0" (at 245.11 81.28 90)
+    (property "Value" "Not used" (at 245.11 81.28 90)
       (effects (font (size 1.27 1.27)) (justify left))
     )
@@
       (effects (font (size 1.27 1.27)) (justify left))
     )
-    (property "Value" "0" (at 220.98 81.28 90)
+    (property "Value" "Not used" (at 220.98 81.28 90)
       (effects (font (size 1.27 1.27)) (justify left))
     )
@@
       (effects (font (size 1.27 1.27)) (justify left))
     )
-    (property "Value" "0" (at 224.79 73.66 90)
+    (property "Value" "Not used" (at 224.79 73.66 90)
       (effects (font (size 1.27 1.27)) (justify left))
     )
@@
       (effects (font (size 1.27 1.27)) (justify left))
     )
-    (property "Value" "0" (at 236.22 81.28 90)
+    (property "Value" "Not used" (at 236.22 81.28 90)
       (effects (font (size 1.27 1.27)) (justify left))
     )
@@
       (effects (font (size 1.27 1.27)) (justify left))
     )
-    (property "Value" "5678uF" (at 391.16 474.98 0)
+    (property "Value" "Not used" (at 391.16 474.98 0)
       (effects (font (size 1.27 1.27)) (justify left))
     )
@@
       (effects (font (size 1.27 1.27)) (justify left))
     )
-    (property "Value" "33pF" (at 572.77 31.75 0)
+    (property "Value" "Not used" (at 572.77 31.75 0)
       (effects (font (size 1.27 1.27)) (justify left))
     )
@@
       (effects (font (size 1.27 1.27)) (justify left))
     )
-    (property "Value" "200pF" (at 476.25 307.34 90)
+    (property "Value" "Not used" (at 476.25 307.34 90)
       (effects (font (size 1.27 1.27)) (justify left))
     )
@@
       (effects (font (size 1.27 1.27)) (justify left))
     )
-    (property "Value" "0" (at 217.17 73.66 90)
+    (property "Value" "Not used" (at 217.17 73.66 90)
       (effects (font (size 1.27 1.27)) (justify left))
     )
@@
       (effects (font (size 1.27 1.27)) (justify left))
     )
-    (property "Value" "0" (at 228.6 81.28 90)
+    (property "Value" "Not used" (at 228.6 81.28 90)
       (effects (font (size 1.27 1.27)) (justify left))
     )

Commit message: Add LCSC part numbers for many devices
Parts:
- C1: LCSC Part # (none) -> C519910
- C14, C2, C24, C25, C27, C3, C30, C38, C39, C4, C40, C43, C44, C45, C49, C5, C50, C51, C52, C54, C6, C7, C8: LCSC Part # (none) -> C519961
- C29, C32, C34, C36: LCSC Part # (none) -> C1854109
- CX1: LCSC Part # (none) -> C520068
- IC16: LCSC Part # (none) -> C10090
- IC19: LCSC Part # (none) -> C2652821
- IC20: LCSC Part # (none) -> C88578
- R1, R2, R6, R7: LCSC Part # (none) -> C17673
- R3: LCSC Part # (none) -> C17520
- R4: LCSC Part # (none) -> C25308
- R5: LCSC Part # (none) -> C25285

Commit message: Add more LCSC part numbers
Parts:
- TR1, TR2: LCSC Part # (none) -> C2891818
Changed lines of the file:
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@@
       (effects (font (size 1.27 1.27)) hide)
     )
-    (property "LCSC Part #" "" (at 530.86 212.09 0)
+    (property "LCSC Part #" "C2891818" (at 530.86 212.09 0)
       (effects (font (size 1.27 1.27)) hide)
     )
@@
       (effects (font (size 1.27 1.27)) hide)
     )
-    (property "LCSC Part #" "" (at 544.83 220.98 0)
-      (effects (font (size 1.27 1.27)) hide)
-    )
+    (property "LCSC Part #" "C2891818" (at 544.83 220.98 0)
+      (effects (font (size 1.27 1.27)) hide)
+    )

Commit message: Add LCSC part number and datasheet for the 10uF SMD caps
Parts:
- C10, C11, C12, C13, C23, C28, C31, C37, C41, C42, C46, C53, C9: LCSC Part # (none) -> C178496
Changed lines of the file:
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@@
       (effects (font (size 1.27 1.27)) hide)
     )
-    (property "Datasheet" "~" (at 734.06 158.75 0)
+    (property "Datasheet" "https://industrial.panasonic.com/cdbs/www-data/pdf/RDE0000/ABA0000C1145.pdf" (at 734.06 158.75 0)
       (effects (font (size 1.27 1.27)) hide)
     )
-    (property "LCSC Part #" "" (at 734.06 158.75 0)
+    (property "LCSC Part #" "C178496" (at 734.06 158.75 0)
       (effects (font (size 1.27 1.27)) hide)
     )
@@
       (effects (font (size 1.27 1.27)) hide)
     )
-    (property "Datasheet" "~" (at 276.86 549.91 0)
+    (property "Datasheet" "https://industrial.panasonic.com/cdbs/www-data/pdf/RDE0000/ABA0000C1145.pdf" (at 276.86 549.91 0)
       (effects (font (size 1.27 1.27)) hide)
     )
@@
       (effects (font (size 1.27 1.27)) hide)
     )
-    (property "LCSC Part #" "" (at 276.86 549.91 0)
+    (property "LCSC Part #" "C178496" (at 276.86 549.91 0)
       (effects (font (size 1.27 1.27)) hide)
     )
@@
       (effects (font (size 1.27 1.27)) hide)
     )
-    (property "Datasheet" "~" (at 789.94 115.57 0)
+    (property "Datasheet" "https://industrial.panasonic.com/cdbs/www-data/pdf/RDE0000/ABA0000C1145.pdf" (at 789.94 115.57 0)
       (effects (font (size 1.27 1.27)) hide)
     )
-    (property "LCSC Part #" "" (at 789.94 115.57 0)
+    (property "LCSC Part #" "C178496" (at 789.94 115.57 0)
       (effects (font (size 1.27 1.27)) hide)
     )
@@
       (effects (font (size 1.27 1.27)) hide)
     )
-    (property "Datasheet" "~" (at 560.07 288.29 0)
+    (property "Datasheet" "https://industrial.panasonic.com/cdbs/www-data/pdf/RDE0000/ABA0000C1145.pdf" (at 560.07 288.29 0)
       (effects (font (size 1.27 1.27)) hide)
     )
-    (property "LCSC Part #" "" (at 560.07 288.29 0)
+    (property "LCSC Part #" "C178496" (at 560.07 288.29 0)
       (effects (font (size 1.27 1.27)) hide)
     )
@@
       (effects (font (size 1.27 1.27)) hide)
     )
-    (property "Datasheet" "~" (at 330.2 347.98 0)
+    (property "Datasheet" "https://industrial.panasonic.com/cdbs/www-data/pdf/RDE0000/ABA0000C1145.pdf" (at 330.2 347.98 0)
       (effects (font (size 1.27 1.27)) hide)
     )
-    (property "LCSC Part #" "" (at 330.2 347.98 0)
+    (property "LCSC Part #" "C178496" (at 330.2 347.98 0)
       (effects (font (size 1.27 1.27)) hide)
     )
@@
       (effects (font (size 1.27 1.27)) hide)
     )
-    (property "Datasheet" "~" (at 595.63 53.34 0)
+    (property "Datasheet" "https://industrial.panasonic.com/cdbs/www-data/pdf/RDE0000/ABA0000C1145.pdf" (at 595.63 53.34 0)
       (effects (font (size 1.27 1.27)) hide)
     )
-    (property "LCSC Part #" "" (at 595.63 53.34 0)
+    (property "LCSC Part #" "C178496" (at 595.63 53.34 0)
       (effects (font (size 1.27 1.27)) hide)
     )
@@
       (effects (font (size 1.27 1.27)) hide)
     )
-    (property "Datasheet" "~" (at 312.42 142.24 0)
+    (property "Datasheet" "https://industrial.panasonic.com/cdbs/www-data/pdf/RDE0000/ABA0000C1145.pdf" (at 312.42 142.24 0)
       (effects (font (size 1.27 1.27)) hide)
     )
-    (property "LCSC Part #" "" (at 312.42 142.24 0)
+    (property "LCSC Part #" "C178496" (at 312.42 142.24 0)
       (effects (font (size 1.27 1.27)) hide)
     )
@@
       (effects (font (size 1.27 1.27)) hide)
     )
-    (property "Datasheet" "~" (at 373.38 67.31 0)
+    (property "Datasheet" "https://industrial.panasonic.com/cdbs/www-data/pdf/RDE0000/ABA0000C1145.pdf" (at 373.38 67.31 0)
       (effects (font (size 1.27 1.27)) hide)
     )
-    (property "LCSC Part #" "" (at 373.38 67.31 0)
+    (property "LCSC Part #" "C178496" (at 373.38 67.31 0)
       (effects (font (size 1.27 1.27)) hide)
     )
@@
       (effects (font (size 1.27 1.27)) hide)
     )
-    (property "Datasheet" "~" (at 248.92 347.98 0)
+    (property "Datasheet" "https://industrial.panasonic.com/cdbs/www-data/pdf/RDE0000/ABA0000C1145.pdf" (at 248.92 347.98 0)
       (effects (font (size 1.27 1.27)) hide)
     )
-    (property "LCSC Part #" "" (at 248.92 347.98 0)
+    (property "LCSC Part #" "C178496" (at 248.92 347.98 0)
       (effects (font (size 1.27 1.27)) hide)
     )
@@
       (effects (font (size 1.27 1.27)) hide)
     )
-    (property "Datasheet" "~" (at 60.96 222.25 0)
+    (property "Datasheet" "https://industrial.panasonic.com/cdbs/www-data/pdf/RDE0000/ABA0000C1145.pdf" (at 60.96 222.25 0)
       (effects (font (size 1.27 1.27)) hide)
     )
-    (property "LCSC Part #" "" (at 60.96 222.25 0)
+    (property "LCSC Part #" "C178496" (at 60.96 222.25 0)
       (effects (font (size 1.27 1.27)) hide)
     )
@@
       (effects (font (size 1.27 1.27)) hide)
     )
-    (property "Datasheet" "~" (at 373.38 142.24 0)
+    (property "Datasheet" "https://industrial.panasonic.com/cdbs/www-data/pdf/RDE0000/ABA0000C1145.pdf" (at 373.38 142.24 0)
       (effects (font (size 1.27 1.27)) hide)
     )
-    (property "LCSC Part #" "" (at 373.38 142.24 0)
+    (property "LCSC Part #" "C178496" (at 373.38 142.24 0)
       (effects (font (size 1.27 1.27)) hide)
     )
@@
       (effects (font (size 1.27 1.27)) hide)
     )
-    (property "Datasheet" "~" (at 312.42 67.31 0)
+    (property "Datasheet" "https://industrial.panasonic.com/cdbs/www-data/pdf/RDE0000/ABA0000C1145.pdf" (at 312.42 67.31 0)
       (effects (font (size 1.27 1.27)) hide)
     )
-    (property "LCSC Part #" "" (at 312.42 67.31 0)
+    (property "LCSC Part #" "C178496" (at 312.42 67.31 0)
       (effects (font (size 1.27 1.27)) hide)
     )
@@
       (effects (font (size 1.27 1.27)) hide)
     )
-    (property "Datasheet" "~" (at 74.93 285.75 0)
+    (property "Datasheet" "https://industrial.panasonic.com/cdbs/www-data/pdf/RDE0000/ABA0000C1145.pdf" (at 74.93 285.75 0)
       (effects (font (size 1.27 1.27)) hide)
     )
-    (property "LCSC Part #" "" (at 74.93 285.75 0)
+    (property "LCSC Part #" "C178496" (at 74.93 285.75 0)
       (effects (font (size 1.27 1.27)) hide)
     )

Commit message: Add MPN field and fill it in
Parts:
- C10, C11, C12, C13, C23, C28, C31, C37, C41, C42, C46, C53, C9: MPN (none) -> EEE1CA100SR
- IC16: MPN (none) -> SN74HC00DR
- IC19: MPN (none) -> SN74HC112DR
- IC20: MPN (none) -> SN74HC245NSR
- TR1, TR2: MPN (none) -> 2SC1623
